File: AVR-CTF/MCU.sch (KiCad schematic (older format))
At the start: 39 parts

Commit message: Esquematico para revision
Parts:
- added J6, J8: Conn_02x07_Counter_Clockwise, Connector_PinHeader_2.54mm:PinHeader_2x07_P2.54mm_Vertical, symbol Connector_Generic:Conn_02x07_Counter_Clockwise
- D5: renamed from D?; value D_Schottky -> SSA14
- gave numbers to parts that had none: 37
Connections:
- net labels added: T_MCU_RX, T_MCU_SCL, T_MCU_SDA, T_MCU_TX
- net labels removed: MONITOR_RX, MONITOR_TX
- wire segments 185 -> 218
Other:
- note added: "F-RAM"
- note added: "HEADERS"
- note added: "MICROCONTROLLER"
- note added: "UPDI PROGRAMMING\n"
- note added: "USB TO TTL"
- moved on the sheet: C11, C12, J4, J5, J7, R6, R9, U4, Y1

Commit message: Versión para revisión
Parts:
- removed J6, J8: Conn_02x07_Counter_Clockwise, Connector_PinHeader_2.54mm:PinHeader_2x07_P2.54mm_Vertical, symbol Connector_Generic:Conn_02x07_Counter_Clockwise
- added D9: COM-11821, AVR-CTF-footprints:LED_COM-11821, symbol AVR-CTF-symbols:COM-11821
- J4, J5: footprint (none) -> Connector_PinHeader_2.54mm:PinHeader_1x02_P2.54mm_Vertical
- J7: footprint (none) -> Connector_PinHeader_2.54mm:PinHeader_1x03_P2.54mm_Vertical
- J9: footprint GCT_USB3090-XX-X_REVE -> AVR-CTF-footprints:GCT_USB3090-XX-X_REVE
Connections:
- net labels added: LED_RGB_DATA
- wire segments 218 -> 195
- no-connect marks 13 -> 15
Other:
- note added: "LED RGB"
- note removed: "HEADERS"
Changed lines of the file:
@@
 F 0 "J4" H 900 4850 50  0000 L CNN
 F 1 "Conn_01x02" H 550 4725 50  0000 L CNN
-F 2 "" H 775 4950 50  0001 C CNN
+F 2 "Connector_PinHeader_2.54mm:PinHeader_1x02_P2.54mm_Vertical" H 775 4950 50  0001 C CNN
 F 3 "~" H 775 4950 50  0001 C CNN
 	1    775  4950
@@
 F 0 "J5" H 1825 4925 50  0000 L CNN
 F 1 "Conn_01x02" H 1525 4725 50  0000 L CNN
-F 2 "" H 1725 4950 50  0001 C CNN
+F 2 "Connector_PinHeader_2.54mm:PinHeader_1x02_P2.54mm_Vertical" H 1725 4950 50  0001 C CNN
 F 3 "~" H 1725 4950 50  0001 C CNN
 	1    1725 4950
@@
 F 0 "J7" H 4368 4500 50  0000 C CNN
 F 1 "Conn_01x03" H 4368 4591 50  0000 C CNN
-F 2 "" H 4450 4825 50  0001 C CNN
+F 2 "Connector_PinHeader_2.54mm:PinHeader_1x03_P2.54mm_Vertical" H 4450 4825 50  0001 C CNN
 F 3 "~" H 4450 4825 50  0001 C CNN
 	1    4450 4825
@@
 F 0 "J9" H 10850 5450 50  0000 L CNN
 F 1 "USB3090-XX-X_REVE" H 10375 5550 50  0001 L CNN
-F 2 "GCT_USB3090-XX-X_REVE" H 10950 4950 50  0001 L BNN
+F 2 "AVR-CTF-footprints:GCT_USB3090-XX-X_REVE" H 10950 4950 50  0001 L BNN
 F 3 "" H 10950 4950 50  0001 L BNN
 F 4 "GCT" H 10950 4950 50  0001 L BNN "MANUFACTURER"
@@
 	8050 2525 7900 2525
 Connection ~ 8050 2525
-$Comp
-L Connector_Generic:Conn_02x07_Counter_Clockwise J6
-U 1 1 622DD113
-P 3900 5975
-F 0 "J6" H 3950 6400 50  0000 C CNN
-F 1 "Conn_02x07_Counter_Clockwise" H 3950 6401 50  0001 C CNN
-F 2 "Connector_PinHeader_2.54mm:PinHeader_2x07_P2.54mm_Vertical" H 3900 5975 50  0001 C CNN
-F 3 "~" H 3900 5975 50  0001 C CNN
-	1    3900 5975
-	1    0    0    -1
-$EndComp
-$Comp
-L Connector_Generic:Conn_02x07_Counter_Clockwise J8
-U 1 1 622DE440
-P 5350 5975
-F 0 "J8" H 5400 6400 50  0000 C CNN
-F 1 "Conn_02x07_Counter_Clockwise" H 5400 6401 50  0001 C CNN
-F 2 "Connector_PinHeader_2.54mm:PinHeader_2x07_P2.54mm_Vertical" H 5350 5975 50  0001 C CNN
-F 3 "~" H 5350 5975 50  0001 C CNN
-	1    5350 5975
-	1    0    0    -1
-$EndComp
-Text GLabel 3450 5775 0    50   Input ~ 0
-PA0
-Wire Wire Line
-	3450 5775 3700 5775
-Text GLabel 3450 5875 0    50   Input ~ 0
-PA1
-Text GLabel 3450 5975 0    50   Input ~ 0
-PA2
-Text GLabel 3450 6075 0    50   Input ~ 0
-PA3
-Text GLabel 3450 6175 0    50   Input ~ 0
-PA4
-Text GLabel 3450 6275 0    50   Input ~ 0
-PA5
-Wire Wire Line
-	3450 5875 3700 5875
-Wire Wire Line
-	3450 5975 3700 5975
-Wire Wire Line
-	3450 6075 3700 6075
-Wire Wire Line
-	3450 6175 3700 6175
-Wire Wire Line
-	3450 6275 3700 6275
-Wire Wire Line
-	4200 6275 4450 6275
-Text GLabel 4450 6275 2    50   Input ~ 0
-PA6
-Wire Wire Line
-	4200 6175 4450 6175
-Text GLabel 4450 6175 2    50   Input ~ 0
-PA7
-Text GLabel 4450 6075 2    50   Input ~ 0
-PF0
-Text GLabel 4450 5875 2    50   Input ~ 0
-PF2
-Text GLabel 4450 5775 2    50   Input ~ 0
-PF3
-Text GLabel 4900 5775 0    50   Input ~ 0
-PF4
-Text GLabel 4900 5875 0    50   Input ~ 0
-PF5
-Wire Wire Line
-	4450 6075 4200 6075
-Wire Wire Line
-	4200 5975 4450 5975
-Wire Wire Line
-	4450 5875 4200 5875
-Wire Wire Line
-	4450 5775 4200 5775
-Wire Wire Line
-	3700 5675 3575 5675
-$Comp
-L power:GND #PWR035
-U 1 1 6239C8BA
-P 4325 5600
-F 0 "#PWR035" H 4325 5350 50  0001 C CNN
-F 1 "GND" H 4250 5600 50  0000 R CNN
-F 2 "" H 4325 5600 50  0001 C CNN
-F 3 "" H 4325 5600 50  0001 C CNN
-	1    4325 5600
-	-1   0    0    1
-$EndComp
-Wire Wire Line
-	4200 5675 4325 5675
-Wire Wire Line
-	4325 5675 4325 5600
-Wire Wire Line
-	5150 5775 4900 5775
-Text GLabel 4450 5975 2    50   Input ~ 0
-PF1
-Wire Wire Line
-	4900 5875 5150 5875
-Text GLabel 4900 5975 0    50   Input ~ 0
-PC0
-Text GLabel 4900 6075 0    50   Input ~ 0
-PC1
-Text GLabel 4900 6175 0    50   Input ~ 0
-PC2
-Text GLabel 4900 6275 0    50   Input ~ 0
-PC3
-Wire Wire Line
-	4900 5975 5150 5975
-Wire Wire Line
-	4900 6075 5150 6075
-Wire Wire Line
-	4900 6175 5150 6175
-Wire Wire Line
-	4900 6275 5150 6275
-Text GLabel 5900 6275 2    50   Input ~ 0
-PD0
-Text GLabel 5900 6175 2    50   Input ~ 0
-PD1
-Text GLabel 5900 6075 2    50   Input ~ 0
-PD2
-Text GLabel 5900 5975 2    50   Input ~ 0
-PD3
-Text GLabel 5900 5875 2    50   Input ~ 0
-PD4
-Text GLabel 5900 5775 2    50   Input ~ 0
-PD5
-Text GLabel 5900 5675 2    50   Input ~ 0
-PD6
-Text GLabel 4900 5675 0    50   Input ~ 0
-PD7
-Wire Wire Line
-	5900 5775 5650 5775
-Wire Wire Line
-	5650 5875 5900 5875
-Wire Wire Line
-	5650 5975 5900 5975
-Wire Wire Line
-	5650 6075 5900 6075
-Wire Wire Line
-	5650 6175 5900 6175
-Wire Wire Line
-	5650 6275 5900 6275
-Wire Wire Line
-	5650 5675 5900 5675
-Wire Wire Line
-	4900 5675 5150 5675
-$Comp
-L power:+3.3V #PWR?
-U 1 1 624BAA86
-P 3575 5675
-AR Path="/621FA25F/624BAA86" Ref="#PWR?"  Part="1"
-AR Path="/6220499D/624BAA86" Ref="#PWR033"  Part="1"
-F 0 "#PWR033" H 3575 5525 50  0001 C CNN
-F 1 "+3.3V" H 3590 5848 50  0000 C CNN
-F 2 "" H 3575 5675 50  0001 C CNN
-F 3 "" H 3575 5675 50  0001 C CNN
-	1    3575 5675
-	1    0    0    -1
-$EndComp
 Wire Notes Line
 	500  5200 500  500
@@
 	7650 2050 8500 2050
 Wire Notes Line
-	3150 5250 3150 6650
-Wire Notes Line
-	3150 6650 6150 6650
-Wire Notes Line
-	6150 6650 6150 5250
-Wire Notes Line
-	6150 5250 3150 5250
-Wire Notes Line
 	7100 6500 7100 3950
 Wire Notes Line
@@
 Text Notes 7750 4150 0    63   Italic 13
 USB TO TTL
-Text Notes 4250 5400 0    63   Italic 13
-HEADERS
 Text Notes 600  5400 0    63   Italic 13
 F-RAM
@@
 Wire Wire Line
 	1275 5950 1275 5850
+$Comp
+L AVR-CTF-symbols:COM-11821 D9
+U 1 1 6236EC5C
+P 4300 6300
+F 0 "D9" H 4450 6765 50  0000 C CNN
+F 1 "COM-11821" H 4450 6674 50  0000 C CNN
+F 2 "AVR-CTF-footprints:LED_COM-11821" H 4035 5720 50  0001 L BNN
+F 3 "" H 4300 6300 50  0001 L BNN
+F 4 "Sparkfun" H 4470 5930 50  0001 L BNN "MANUFACTURER"
+F 5 "Manufacturer recommendations" H 3790 5815 50  0001 L BNN "STANDARD"
+	1    4300 6300
+	1    0    0    -1
+$EndComp
+$Comp
+L power:+5V #PWR013
+U 1 1 623717DB
+P 5100 6100
+F 0 "#PWR013" H 5100 5950 50  0001 C CNN
+F 1 "+5V" H 5115 6273 50  0000 C CNN
+F 2 "" H 5100 6100 50  0001 C CNN
+F 3 "" H 5100 6100 50  0001 C CNN
+	1    5100 6100
+	1    0    0    -1
+$EndComp
+Wire Wire Line
+	4900 6200 5100 6200
+Wire Wire Line
+	5100 6200 5100 6100
+$Comp
+L power:GND #PWR016
+U 1 1 6237E339
+P 5100 6550
+F 0 "#PWR016" H 5100 6300 50  0001 C CNN
+F 1 "GND" H 5300 6550 50  0000 R CNN
+F 2 "" H 5100 6550 50  0001 C CNN
+F 3 "" H 5100 6550 50  0001 C CNN
+	1    5100 6550
+	1    0    0    -1
+$EndComp
+Wire Wire Line
+	4900 6400 5100 6400
+Wire Wire Line
+	5100 6400 5100 6550
+Wire Wire Line
+	4000 6200 3500 6200
+Text Label 3500 6200 0    50   ~ 0
+LED_RGB_DATA
+NoConn ~ 4900 6300
+NoConn ~ 4900 6100
+Text Label 4550 5650 0    50   ~ 0
+LED_RGB_DATA
+Wire Wire Line
+	4550 5650 4200 5650
+Wire Notes Line
+	3150 5250 5400 5250
+Wire Notes Line
+	5400 5250 5400 6700
+Wire Notes Line
+	5400 6700 3150 6700
+Wire Notes Line
+	3150 6700 3150 5250
+Text Notes 4150 5450 0    63   Italic 13
+LED RGB
+Text GLabel 4200 5650 0    50   Input ~ 0
+PD0
 $EndSCHEMATC

Commit message: Correciones del retorno de tierra
Connections:
- net labels added: VDD
- net labels removed: GND1
Changed lines of the file:
@@
 	3600 3475 3600 3575
-$Comp
-L power:GND1 #PWR034
-U 1 1 62207FD2
-P 3600 3775
-F 0 "#PWR034" H 3600 3525 50  0001 C CNN
-F 1 "GND1" H 3605 3602 50  0000 C CNN
-F 2 "" H 3600 3775 50  0001 C CNN
-F 3 "" H 3600 3775 50  0001 C CNN
-	1    3600 3775
-	1    0    0    -1
-$EndComp
 $Comp
 L pspice:INDUCTOR L1
@@
 $Comp
 L power:+3.3V #PWR?
-U 1 1 6220D2E2
-P 2325 3275
-AR Path="/621FA25F/6220D2E2" Ref="#PWR?"  Part="1"
-AR Path="/6220499D/6220D2E2" Ref="#PWR031"  Part="1"
-F 0 "#PWR031" H 2325 3125 50  0001 C CNN
-F 1 "+3.3V" H 2340 3448 50  0000 C CNN
-F 2 "" H 2325 3275 50  0001 C CNN
-F 3 "" H 2325 3275 50  0001 C CNN
-	1    2325 3275
-	1    0    0    -1
-$EndComp
-$Comp
-L power:+3.3V #PWR?
 U 1 1 6222DF18
 P 1275 2250
@@
 F 3 "" H 1275 2250 50  0001 C CNN
 	1    1275 2250
-	1    0    0    -1
-$EndComp
-$Comp
-L power:GND1 #PWR028
-U 1 1 6222E76E
-P 1275 2950
-F 0 "#PWR028" H 1275 2700 50  0001 C CNN
-F 1 "GND1" H 1280 2777 50  0000 C CNN
-F 2 "" H 1275 2950 50  0001 C CNN
-F 3 "" H 1275 2950 50  0001 C CNN
-	1    1275 2950
 	1    0    0    -1
 $EndComp
@@
 UPDI
 $Comp
-L power:GND1 #PWR037
-U 1 1 622C141B
-P 5050 4925
-F 0 "#PWR037" H 5050 4675 50  0001 C CNN
-F 1 "GND1" H 5055 4752 50  0000 C CNN
-F 2 "" H 5050 4925 50  0001 C CNN
-F 3 "" H 5050 4925 50  0001 C CNN
-	1    5050 4925
-	1    0    0    -1
-$EndComp
-$Comp
 L power:+3.3V #PWR?
 U 1 1 622C166B
@@
 	800  3150 800  3200
 Wire Wire Line
-	800  3200 900  3200
-Wire Wire Line
 	1000 3200 1000 3150
 Wire Wire Line
 	1275 2900 1275 2950
-$Comp
-L power:GND1 #PWR023
-U 1 1 622D9C91
-P 900 3200
-F 0 "#PWR023" H 900 2950 50  0001 C CNN
-F 1 "GND1" H 905 3027 50  0000 C CNN
-F 2 "" H 900 3200 50  0001 C CNN
-F 3 "" H 900 3200 50  0001 C CNN
-	1    900  3200
-	1    0    0    -1
-$EndComp
-Connection ~ 900  3200
-Wire Wire Line
-	900  3200 1000 3200
 $Comp
 L AVR-CTF-symbols:4-1437565-2 SW?
@@
 	950  1775 950  1825
 Wire Wire Line
-	950  1825 1050 1825
-Wire Wire Line
 	1150 1825 1150 1775
 Wire Wire Line
@@
 Wire Wire Line
 	1050 875  1050 925
-$Comp
-L power:GND1 #PWR025
-U 1 1 622FD944
-P 1050 1825
-F 0 "#PWR025" H 1050 1575 50  0001 C CNN
-F 1 "GND1" H 1055 1652 50  0000 C CNN
-F 2 "" H 1050 1825 50  0001 C CNN
-F 3 "" H 1050 1825 50  0001 C CNN
-	1    1050 1825
-	1    0    0    -1
-$EndComp
-Connection ~ 1050 1825
-Wire Wire Line
-	1050 1825 1150 1825
 Wire Wire Line
 	1275 1225 1150 1225
@@
 Boot
 $Comp
-L power:GND1 #PWR043
-U 1 1 62417937
-P 8400 2350
-F 0 "#PWR043" H 8400 2100 50  0001 C CNN
-F 1 "GND1" H 8405 2177 50  0000 C CNN
-F 2 "" H 8400 2350 50  0001 C CNN
-F 3 "" H 8400 2350 50  0001 C CNN
-	1    8400 2350
-	1    0    0    -1
-$EndComp
-$Comp
 L power:+3.3V #PWR?
 U 1 1 62479AB7
@@
 Text GLabel 7900 2525 0    50   Input ~ 0
 PA4
-$Comp
-L power:GND1 #PWR040
-U 1 1 6243827D
-P 8250 1800
-F 0 "#PWR040" H 8250 1550 50  0001 C CNN
-F 1 "GND1" H 8255 1627 50  0000 C CNN
-F 2 "" H 8250 1800 50  0001 C CNN
-F 3 "" H 8250 1800 50  0001 C CNN
-	1    8250 1800
-	1    0    0    -1
-$EndComp
 Wire Wire Line
 	8250 1125 8250 1200
@@
 Text GLabel 4200 5650 0    50   Input ~ 0
 PD0
+$Comp
+L power:VDD #PWR0113
+U 1 1 6272FCF8
+P 2325 3275
+F 0 "#PWR0113" H 2325 3125 50  0001 C CNN
+F 1 "VDD" H 2340 3448 50  0000 C CNN
+F 2 "" H 2325 3275 50  0001 C CNN
+F 3 "" H 2325 3275 50  0001 C CNN
+	1    2325 3275
+	1    0    0    -1
+$EndComp
+$Comp
+L power:GND #PWR0114
+U 1 1 627389CC
+P 3600 3775
+F 0 "#PWR0114" H 3600 3525 50  0001 C CNN
+F 1 "GND" H 3800 3775 50  0000 R CNN
+F 2 "" H 3600 3775 50  0001 C CNN
+F 3 "" H 3600 3775 50  0001 C CNN
+	1    3600 3775
+	1    0    0    -1
+$EndComp
+$Comp
+L power:GND #PWR0115
+U 1 1 62738E4B
+P 5050 4925
+F 0 "#PWR0115" H 5050 4675 50  0001 C CNN
+F 1 "GND" H 5250 4925 50  0000 R CNN
+F 2 "" H 5050 4925 50  0001 C CNN
+F 3 "" H 5050 4925 50  0001 C CNN
+	1    5050 4925
+	1    0    0    -1
+$EndComp
+$Comp
+L power:GND #PWR0116
+U 1 1 627394B9
+P 1275 2950
+F 0 "#PWR0116" H 1275 2700 50  0001 C CNN
+F 1 "GND" H 1475 2950 50  0000 R CNN
+F 2 "" H 1275 2950 50  0001 C CNN
+F 3 "" H 1275 2950 50  0001 C CNN
+	1    1275 2950
+	1    0    0    -1
+$EndComp
+Wire Wire Line
+	800  3200 900  3200
+$Comp
+L power:GND #PWR0117
+U 1 1 627398B1
+P 900 3200
+F 0 "#PWR0117" H 900 2950 50  0001 C CNN
+F 1 "GND" H 1100 3200 50  0000 R CNN
+F 2 "" H 900 3200 50  0001 C CNN
+F 3 "" H 900 3200 50  0001 C CNN
+	1    900  3200
+	1    0    0    -1
+$EndComp
+Connection ~ 900  3200
+Wire Wire Line
+	900  3200 1000 3200
+$Comp
+L power:GND #PWR0118
+U 1 1 62739B29
+P 1045 1825
+F 0 "#PWR0118" H 1045 1575 50  0001 C CNN
+F 1 "GND" H 1240 1730 50  0000 R CNN
+F 2 "" H 1045 1825 50  0001 C CNN
+F 3 "" H 1045 1825 50  0001 C CNN
+	1    1045 1825
+	1    0    0    -1
+$EndComp
+Wire Wire Line
+	950  1825 1045 1825
+Connection ~ 1045 1825
+Wire Wire Line
+	1045 1825 1150 1825
+$Comp
+L power:GND #PWR?
+U 1 1 62751097
+P 8250 1800
+F 0 "#PWR?" H 8250 1550 50  0001 C CNN
+F 1 "GND" H 8330 1650 50  0000 R CNN
+F 2 "" H 8250 1800 50  0001 C CNN
+F 3 "" H 8250 1800 50  0001 C CNN
+	1    8250 1800
+	1    0    0    -1
+$EndComp
+$Comp
+L power:GND #PWR?
+U 1 1 62751E24
+P 8400 2350
+F 0 "#PWR?" H 8400 2100 50  0001 C CNN
+F 1 "GND" H 8480 2200 50  0000 R CNN
+F 2 "" H 8400 2350 50  0001 C CNN
+F 3 "" H 8400 2350 50  0001 C CNN
+	1    8400 2350
+	1    0    0    -1
+$EndComp
 $EndSCHEMATC
