File: AVR-CTF/MCU.sch (KiCad schematic (older format))
At the start: 39 parts, among them J4 Conn_01x02, J5 Conn_01x02, J7 Conn_01x03, J9 USB3090-XX-X_REVE, P1 Power, P2 Analog, P3 Digital, P4 Digital, SW3 4-1437565-2, SW4 4-1437565-2, SW5 4-1437565-2, U4 FM24C04B-GTR, U5 AVR32DA32-I_PT, U6 CY7C65211-24LTXI, Y1 ABS07

Commit message: Generacion .cache 2
Parts:
- renumbered C11 to C16, C12 to C17, C13 to C18, C14 to C19, C15 to C20, C16 to C21, C17 to C22, C18 to C23, C19 to C24, D9 to D5, D2 to D6, D3 to D7, D4 to D8, D5 to D9, J4 to J5, J5 to J6, J9 to J8, R6 to R11, R7 to R12, R8 to R13, R9 to R14, R10 to R15, R11 to R16, R12 to R17, R13 to R18, R14 to R19, U4 to U6, U5 to U7, U6 to U8
