File: AVR-CTF/MONITOR.sch (KiCad schematic (older format))
At the start: 24 parts, among them J10 USB3090-XX-X_REVE, J3 Prog, SW1 4-1437565-2, SW2 4-1437565-2, U3 ESP32-WROOM-32D, U9 CY7C65211-24LTXI

Commit message: Generacion .cache 2
Parts:
- renumbered C24 to C10, C8 to C11, C9 to C12, C25 to C13, C26 to C14, C27 to C15, C6 to C8, C7 to C9, D6 to D2, D7 to D3, D8 to D4, J10 to J4, R17 to R10, R2 to R4, R3 to R5, R15 to R6, R4 to R7, R5 to R8, R16 to R9, U3 to U4, U9 to U5
