File: AVR-CTF/power_supply.sch (KiCad schematic (older format))
At the start: 16 parts, among them J1 Conn_01x02, J2 Conn_01x03, U1 AMS1117-5.0, U2 AMS1117-3.3, U7 AMS1117-3.3

Commit message: Correciones del retorno de tierra
Connections:
- net labels added: +3V3, VDD
- net labels removed: +3.3V, GND1
Changed lines of the file:
@@
 3.3V POWER SUPPLY
-$Comp
-L power:+3.3V #PWR07
-U 1 1 6210133B
-P 2750 3075
-F 0 "#PWR07" H 2750 2925 50  0001 C CNN
-F 1 "+3.3V" H 2765 3248 50  0000 C CNN
-F 2 "" H 2750 3075 50  0001 C CNN
-F 3 "" H 2750 3075 50  0001 C CNN
-	1    2750 3075
-	1    0    0    -1
-$EndComp
-Connection ~ 2750 3075
 $Comp
 L power:+5V #PWR04
@@
 POWER LED
 $Comp
-L power:GND #PWR?
-U 1 1 621350E1
-P 4400 1950
-AR Path="/621350E1" Ref="#PWR?"  Part="1"
-AR Path="/620E3406/621350E1" Ref="#PWR011"  Part="1"
-AR Path="/621FA25F/621350E1" Ref="#PWR09"  Part="1"
-F 0 "#PWR09" H 4400 1700 50  0001 C CNN
-F 1 "GND" H 4475 1775 50  0000 R CNN
-F 2 "" H 4400 1950 50  0001 C CNN
-F 3 "" H 4400 1950 50  0001 C CNN
-	1    4400 1950
-	1    0    0    -1
-$EndComp
-$Comp
 L Connector_Generic:Conn_01x02 J?
 U 1 1 621350E7
@@
 Wire Wire Line
 	4400 1900 4400 1950
-$Comp
-L power:GND1 #PWR010
-U 1 1 6220336F
-P 4625 1950
-F 0 "#PWR010" H 4625 1700 50  0001 C CNN
-F 1 "GND1" H 4630 1777 50  0000 C CNN
-F 2 "" H 4625 1950 50  0001 C CNN
-F 3 "" H 4625 1950 50  0001 C CNN
-	1    4625 1950
-	1    0    0    -1
-$EndComp
 Wire Wire Line
 	4625 1950 4625 1800
@@
 Wire Notes Line
 	1750 4975 1750 3825
-$Comp
-L power:+3.3V #PWR012
-U 1 1 627A1439
-P 3700 4400
-F 0 "#PWR012" H 3700 4250 50  0001 C CNN
-F 1 "+3.3V" H 3715 4573 50  0000 C CNN
-F 2 "" H 3700 4400 50  0001 C CNN
-F 3 "" H 3700 4400 50  0001 C CNN
-	1    3700 4400
-	1    0    0    -1
-$EndComp
 $Comp
 L Device:R R?
@@
 $EndComp
 Wire Wire Line
-	2570 4400 2550 4400
-Wire Wire Line
 	2250 4400 2220 4400
 $Comp
@@
 AR Path="/620E3406/6235288C" Ref="R?"  Part="1"
 AR Path="/621FA25F/6235288C" Ref="R19"  Part="1"
-F 0 "R19" V 3390 4310 50  0000 C CNN
+F 0 "R19" V 3275 4385 50  0000 C CNN
 F 1 "0" V 3390 4390 50  0000 C CNN
 F 2 "Resistor_SMD:R_0603_1608Metric_Pad0.98x0.95mm_HandSolder" V 3420 4400 50  0001 C CNN
@@
 Wire Wire Line
 	3640 4400 3700 4400
+$Comp
+L power:+3V3 #PWR0109
+U 1 1 6271A86D
+P 4625 1950
+F 0 "#PWR0109" H 4625 1800 50  0001 C CNN
+F 1 "+3V3" H 4640 2123 50  0000 C CNN
+F 2 "" H 4625 1950 50  0001 C CNN
+F 3 "" H 4625 1950 50  0001 C CNN
+	1    4625 1950
+	-1   0    0    1
+$EndComp
+$Comp
+L power:+3V3 #PWR0110
+U 1 1 62730BD7
+P 2750 3075
+F 0 "#PWR0110" H 2750 2925 50  0001 C CNN
+F 1 "+3V3" H 2765 3248 50  0000 C CNN
+F 2 "" H 2750 3075 50  0001 C CNN
+F 3 "" H 2750 3075 50  0001 C CNN
+	1    2750 3075
+	1    0    0    -1
+$EndComp
+Connection ~ 2750 3075
+$Comp
+L power:+3V3 #PWR0111
+U 1 1 6273127A
+P 3700 4400
+F 0 "#PWR0111" H 3700 4250 50  0001 C CNN
+F 1 "+3V3" H 3715 4573 50  0000 C CNN
+F 2 "" H 3700 4400 50  0001 C CNN
+F 3 "" H 3700 4400 50  0001 C CNN
+	1    3700 4400
+	1    0    0    -1
+$EndComp
 Connection ~ 3700 4400
+$Comp
+L power:VDD #PWR0112
+U 1 1 6273201F
+P 4400 1950
+F 0 "#PWR0112" H 4400 1800 50  0001 C CNN
+F 1 "VDD" H 4415 2123 50  0000 C CNN
+F 2 "" H 4400 1950 50  0001 C CNN
+F 3 "" H 4400 1950 50  0001 C CNN
+	1    4400 1950
+	-1   0    0    1
+$EndComp
+Wire Wire Line
+	2550 4400 2575 4400
 $EndSCHEMATC

Commit message: Generacion .cache 2
Parts:
- renumbered C20 to C6, C21 to C7, D3 to D1, R2 to R1, R18 to R2, R19 to R3, U7 to U3
Changed lines of the file:
@@
 P 4375 3175
 AR Path="/621106C5" Ref="#PWR?"  Part="1"
-AR Path="/620E3406/621106C5" Ref="#PWR010"  Part="1"
-AR Path="/621FA25F/621106C5" Ref="#PWR08"  Part="1"
-F 0 "#PWR08" H 4375 3025 50  0001 C CNN
+AR Path="/620E3406/621106C5" Ref="#PWR?"  Part="1"
+AR Path="/621FA25F/621106C5" Ref="#PWR011"  Part="1"
+F 0 "#PWR011" H 4375 3025 50  0001 C CNN
 F 1 "+5V" V 4350 3350 50  0000 C CNN
 F 2 "" H 4375 3175 50  0001 C CNN
@@
 P 4175 3175
 AR Path="/621106CB" Ref="J?"  Part="1"
-AR Path="/620E3406/621106CB" Ref="J2"  Part="1"
+AR Path="/620E3406/621106CB" Ref="J?"  Part="1"
 AR Path="/621FA25F/621106CB" Ref="J2"  Part="1"
 F 0 "J2" H 4093 3492 50  0000 C CNN
@@
 P 1175 4675
 AR Path="/6211D42D" Ref="D?"  Part="1"
-AR Path="/620E3406/6211D42D" Ref="D3"  Part="1"
+AR Path="/620E3406/6211D42D" Ref="D?"  Part="1"
 AR Path="/621FA25F/6211D42D" Ref="D1"  Part="1"
 F 0 "D1" V 1168 4892 50  0000 C CNN
@@
 P 1175 4375
 AR Path="/6211D433" Ref="R?"  Part="1"
-AR Path="/620E3406/6211D433" Ref="R2"  Part="1"
+AR Path="/620E3406/6211D433" Ref="R?"  Part="1"
 AR Path="/621FA25F/6211D433" Ref="R1"  Part="1"
 F 0 "R1" H 968 4375 50  0000 C CNN
@@
 P 1175 4825
 AR Path="/6211D43F" Ref="#PWR?"  Part="1"
-AR Path="/620E3406/6211D43F" Ref="#PWR07"  Part="1"
+AR Path="/620E3406/6211D43F" Ref="#PWR?"  Part="1"
 AR Path="/621FA25F/6211D43F" Ref="#PWR02"  Part="1"
 F 0 "#PWR02" H 1175 4575 50  0001 C CNN
@@
 P 4125 1900
 AR Path="/621350E7" Ref="J?"  Part="1"
-AR Path="/620E3406/621350E7" Ref="J1"  Part="1"
+AR Path="/620E3406/621350E7" Ref="J?"  Part="1"
 AR Path="/621FA25F/621350E7" Ref="J1"  Part="1"
 F 0 "J1" H 4043 1575 50  0000 C CNN
@@
 	4325 1800 4625 1800
 $Comp
-L power:+5V #PWR0105
+L power:+5V #PWR01
 U 1 1 62750FD7
 P 1175 4225
-F 0 "#PWR0105" H 1175 4075 50  0001 C CNN
+F 0 "#PWR01" H 1175 4075 50  0001 C CNN
 F 1 "+5V" H 1175 4400 50  0000 C CNN
 F 2 "" H 1175 4225 50  0001 C CNN
@@
 Connection ~ 2875 4700
 $Comp
-L power:GND #PWR011
+L power:GND #PWR09
 U 1 1 6278C8CD
 P 2875 4700
-F 0 "#PWR011" H 2875 4450 50  0001 C CNN
+F 0 "#PWR09" H 2875 4450 50  0001 C CNN
 F 1 "GND" H 2880 4527 50  0000 C CNN
 F 2 "" H 2875 4700 50  0001 C CNN
@@
 	3175 4400 3250 4400
 $Comp
-L Device:C C21
+L Device:C C7
 U 1 1 6278C8D9
 P 3700 4550
-F 0 "C21" H 3815 4596 50  0000 L CNN
+F 0 "C7" H 3815 4596 50  0000 L CNN
 F 1 "10uF" H 3815 4505 50  0000 L CNN
 F 2 "Capacitor_SMD:C_0603_1608Metric_Pad1.08x0.95mm_HandSolder" H 3738 4400 50  0001 C CNN
@@
 $EndComp
 $Comp
-L Device:CP C20
+L Device:CP C6
 U 1 1 6278C8DF
 P 3250 4550
-F 0 "C20" H 3368 4596 50  0000 L CNN
+F 0 "C6" H 3368 4596 50  0000 L CNN
 F 1 "10uF" H 3368 4505 50  0000 L CNN
 F 2 "Capacitor_SMD:C_0805_2012Metric_Pad1.18x1.45mm_HandSolder" H 3288 4400 50  0001 C CNN
@@
 $EndComp
 $Comp
-L Regulator_Linear:AMS1117-3.3 U7
+L Regulator_Linear:AMS1117-3.3 U3
 U 1 1 6278C8E6
 P 2875 4400
-F 0 "U7" H 2875 4642 50  0000 C CNN
+F 0 "U3" H 2875 4642 50  0000 C CNN
 F 1 "AMS1117-3.3" H 2875 4551 50  0000 C CNN
 F 2 "Package_TO_SOT_SMD:SOT-223-3_TabPin2" H 2875 4600 50  0001 C CNN
@@
 ESP POWER SUPPLY
 $Comp
-L power:+5V #PWR01
+L power:+5V #PWR07
 U 1 1 6278C8F4
 P 2220 4400
-F 0 "#PWR01" H 2220 4250 50  0001 C CNN
+F 0 "#PWR07" H 2220 4250 50  0001 C CNN
 F 1 "+5V" H 2220 4575 50  0000 C CNN
 F 2 "" H 2220 4400 50  0001 C CNN
@@
 AR Path="/62350913" Ref="R?"  Part="1"
 AR Path="/620E3406/62350913" Ref="R?"  Part="1"
-AR Path="/621FA25F/62350913" Ref="R18"  Part="1"
-F 0 "R18" V 2500 4400 50  0000 C CNN
+AR Path="/621FA25F/62350913" Ref="R2"  Part="1"
+F 0 "R2" V 2500 4400 50  0000 C CNN
 F 1 "0" V 2300 4390 50  0000 C CNN
 F 2 "Resistor_SMD:R_0603_1608Metric_Pad0.98x0.95mm_HandSolder" V 2330 4400 50  0001 C CNN
@@
 AR Path="/6235288C" Ref="R?"  Part="1"
 AR Path="/620E3406/6235288C" Ref="R?"  Part="1"
-AR Path="/621FA25F/6235288C" Ref="R19"  Part="1"
-F 0 "R19" V 3275 4385 50  0000 C CNN
+AR Path="/621FA25F/6235288C" Ref="R3"  Part="1"
+F 0 "R3" V 3275 4385 50  0000 C CNN
 F 1 "0" V 3390 4390 50  0000 C CNN
 F 2 "Resistor_SMD:R_0603_1608Metric_Pad0.98x0.95mm_HandSolder" V 3420 4400 50  0001 C CNN
@@
 	3640 4400 3700 4400
 $Comp
-L power:+3V3 #PWR0109
+L power:+3V3 #PWR013
 U 1 1 6271A86D
 P 4625 1950
-F 0 "#PWR0109" H 4625 1800 50  0001 C CNN
+F 0 "#PWR013" H 4625 1800 50  0001 C CNN
 F 1 "+3V3" H 4640 2123 50  0000 C CNN
 F 2 "" H 4625 1950 50  0001 C CNN
@@
 $EndComp
 $Comp
-L power:+3V3 #PWR0110
+L power:+3V3 #PWR08
 U 1 1 62730BD7
 P 2750 3075
-F 0 "#PWR0110" H 2750 2925 50  0001 C CNN
+F 0 "#PWR08" H 2750 2925 50  0001 C CNN
 F 1 "+3V3" H 2765 3248 50  0000 C CNN
 F 2 "" H 2750 3075 50  0001 C CNN
@@
 Connection ~ 2750 3075
 $Comp
-L power:+3V3 #PWR0111
+L power:+3V3 #PWR010
 U 1 1 6273127A
 P 3700 4400
-F 0 "#PWR0111" H 3700 4250 50  0001 C CNN
+F 0 "#PWR010" H 3700 4250 50  0001 C CNN
 F 1 "+3V3" H 3715 4573 50  0000 C CNN
 F 2 "" H 3700 4400 50  0001 C CNN
@@
 Connection ~ 3700 4400
 $Comp
-L power:VDD #PWR0112
+L power:VDD #PWR012
 U 1 1 6273201F
 P 4400 1950
-F 0 "#PWR0112" H 4400 1800 50  0001 C CNN
+F 0 "#PWR012" H 4400 1800 50  0001 C CNN
 F 1 "VDD" H 4415 2123 50  0000 C CNN
 F 2 "" H 4400 1950 50  0001 C CNN
